Commit message: Update digit_ysp.urdf

File: digit_ysp.urdf (robot description, URDF)
Before this commit: robot digit, 47 links, 46 joints
Links:
- added link contact1; visual sphere radius=0.015
- added link contact2; visual sphere radius=0.015
- added link contact3; visual sphere radius=0.015
- added link contact4; visual sphere radius=0.015
- added link contact5; visual sphere radius=0.015
- added link contact6; visual sphere radius=0.015
- added link contact7; visual sphere radius=0.015
- added link contact8; visual sphere radius=0.015
- added link cp_left_achillies_rod; visual sphere radius=0.010
- added link cp_left_heel_spring; visual sphere radius=0.015
- added link cp_left_toe_A_rod; visual sphere radius=0.010
- added link cp_left_toe_B_rod; visual sphere radius=0.010
- added link cp_left_toe_roll_A; visual sphere radius=0.015
- added link cp_left_toe_roll_B; visual sphere radius=0.015
- added link cp_right_achillies_rod; visual sphere radius=0.010
- added link cp_right_heel_spring; visual sphere radius=0.015
- added link cp_right_toe_A_rod; visual sphere radius=0.010
- added link cp_right_toe_B_rod; visual sphere radius=0.010
- added link cp_right_toe_roll_A; visual sphere radius=0.015
- added link cp_right_toe_roll_B; visual sphere radius=0.015
Joints:
- added joint contact1_joint: type fixed, parent left_toe_roll, child contact1, origin xyz=0 0 0 rpy=0 0 0
- added joint contact2_joint: type fixed, parent left_toe_roll, child contact2, origin xyz=0 0 0 rpy=0 0 0
- added joint contact3_joint: type fixed, parent left_toe_roll, child contact3, origin xyz=0 0 0 rpy=0 0 0
- added joint contact4_joint: type fixed, parent left_toe_roll, child contact4, origin xyz=0 0 0 rpy=0 0 0
- added joint contact5_joint: type fixed, parent right_toe_roll, child contact5, origin xyz=0 0 0 rpy=0 0 0
- added joint contact6_joint: type fixed, parent right_toe_roll, child contact6, origin xyz=0 0 0 rpy=0 0 0
- added joint contact7_joint: type fixed, parent right_toe_roll, child contact7, origin xyz=0 0 0 rpy=0 0 0
- added joint contact8_joint: type fixed, parent right_toe_roll, child contact8, origin xyz=0 0 0 rpy=0 0 0
- added joint cp_left_achillies_rod_joint: type fixed, parent left_achillies_rod, child cp_left_achillies_rod, origin xyz=0.501194 -1.28948e-05 -5.20307e-06 rpy=0 0 0, axis 0 0 1
- added joint cp_left_heel_spring_joint: type fixed, parent left_heel_spring, child cp_left_heel_spring, origin xyz=0.113789 -0.011056 0 rpy=0 0 0, axis 0 0 1
- added joint cp_left_toe_A_rod_joint: type fixed, parent left_toe_A_rod, child cp_left_toe_A_rod, origin xyz=0.340004 1.61352e-05 -8.14295e-06 rpy=0 0 0, axis 0 0 1
- added joint cp_left_toe_B_rod_joint: type fixed, parent left_toe_B_rod, child cp_left_toe_B_rod, origin xyz=0.288005 -9.72801e-06 -2.23467e-05 rpy=0 0 0, axis 0 0 1
- added joint cp_left_toe_roll_A_joint: type fixed, parent left_toe_roll, child cp_left_toe_roll_A, origin xyz=0.0179 -0.009551 -0.054164 rpy=0 0 0, axis 0 0 1
- added joint cp_left_toe_roll_B_joint: type fixed, parent left_toe_roll, child cp_left_toe_roll_B, origin xyz=-0.0181 -0.009551 -0.054164 rpy=0 0 0, axis 0 0 1
- added joint cp_right_achillies_rod_joint: type fixed, parent right_achillies_rod, child cp_right_achillies_rod, origin xyz=0.501194 -1.28948e-05 -5.20307e-06 rpy=0 0 0, axis 0 0 1
- added joint cp_right_heel_spring_joint: type fixed, parent right_heel_spring, child cp_right_heel_spring, origin xyz=0.113789 0.011056 0 rpy=0 0 0, axis 0 0 1
- added joint cp_right_toe_A_rod_joint: type fixed, parent right_toe_A_rod, child cp_right_toe_A_rod, origin xyz=0.340004 1.61352e-05 -8.14295e-06 rpy=0 0 0, axis 0 0 1
- added joint cp_right_toe_B_rod_joint: type fixed, parent right_toe_B_rod, child cp_right_toe_B_rod, origin xyz=0.288005 -9.72801e-06 -2.23467e-05 rpy=0 0 0, axis 0 0 1
- added joint cp_right_toe_roll_A_joint: type fixed, parent right_toe_roll, child cp_right_toe_roll_A, origin xyz=0.0179 0.009551 -0.054164 rpy=0 0 0, axis 0 0 1
- added joint cp_right_toe_roll_B_joint: type fixed, parent right_toe_roll, child cp_right_toe_roll_B, origin xyz=-0.0181 0.009551 -0.054164 rpy=0 0 0, axis 0 0 1
- joint left_toe_A_rod_parent_joint: origin xyz=0.057 0 -0.008 rpy=-0.037531 0.0046535 -1.6049813 -> xyz=0.057 0 -0.008 rpy=-0.0374899 0.0049742 -1.5964351
- joint left_toe_B_rod_parent_joint: origin xyz=0.057 0 -0.008 rpy=-0.0538329 -0.0025446 1.5948471 -> xyz=0.057 0 -0.008 rpy=-0.0536482 0.0051326 1.5948474
- joint right_elbow_joint: origin xyz=0 -0.0385 0.185 rpy=1.57079632679 -0.3926991 0 -> xyz=0 0.0385 0.185 rpy=-1.57079632679 -0.3926991 0
- joint right_toe_A_rod_parent_joint: origin xyz=0.057 0 -0.008 rpy=0.037531 0.0046535 1.6049813 -> xyz=0.057 0 -0.008 rpy=0.0374899 0.0049742 1.5964351
- joint right_toe_B_rod_parent_joint: origin xyz=0.057 0 -0.008 rpy=0.0538329 -0.0025446 -1.5948471 -> xyz=0.057 0 -0.008 rpy=0.0536482 0.0051326 -1.5948474
- joint shoulder_yaw_joint_right: origin xyz=0 -0.165 -0.1 rpy=1.57079632679 0 0 -> xyz=0 0.165 -0.1 rpy=-1.57079632679 0 0
