Commit message: good version

File: third_party/Task-Space-Control/test/digit_ysp.urdf (robot description, URDF)
Before this commit: robot digit, 61 links, 60 joints
Joints:
- removed joint left_hip_roll_joint
- removed joint right_hip_roll_joint
- added joint left-hip-roll_joint: type revolute, parent torso, child left_hip_roll, origin xyz=-0.001 0.091 0 rpy=1.57079632679 -1.1955506 -1.57079632679, axis 0 0 1, limit lower=-1.0472 upper=1.0472 effort=1.4 velocity=12.15
- added joint right-hip-roll_joint: type revolute, parent torso, child right_hip_roll, origin xyz=-0.001 -0.091 0 rpy=-1.57079632679 -1.1955506 1.57079632679, axis 0 0 1, limit lower=-1.0472 upper=1.0472 effort=1.4 velocity=12.15
