Commit message: add closed loop

File: Simulation/model/digit_ysp.urdf (robot description, URDF)
Before this commit: robot digit, 61 links, 60 joints
Joints:
- joint left_elbow_joint: limit lower=-1.3526 upper=1.3526 effort=1.4 velocity=12.5 -> lower=-1.3526 upper=1.3526 effort=112 velocity=12.5
- joint left_hip_pitch_joint: limit lower=-1.0472 upper=1.57079632679 effort=12.5 velocity=8.5 -> lower=-1.0472 upper=1.57079632679 effort=200 velocity=8.5
- joint left_hip_roll_joint: limit lower=-1.0472 upper=1.0472 effort=1.4 velocity=12.15 -> lower=-1.0472 upper=1.0472 effort=112 velocity=12.15
- joint left_hip_yaw_joint: limit lower=-0.698132 upper=0.698132 effort=1.4 velocity=12.15 -> lower=-0.698132 upper=0.698132 effort=70 velocity=12.15
- joint left_knee_joint: limit lower=-1.2392 upper=0.8727 effort=12.5 velocity=8.5085 -> lower=-1.2392 upper=0.8727 effort=200 velocity=8.5085
- joint left_shoulder_pitch_joint: limit lower=-2.5307 upper=2.5307 effort=1.4 velocity=12.5 -> lower=-2.5307 upper=2.5307 effort=112 velocity=12.5
- joint left_shoulder_roll_joint: limit lower=-1.309 upper=1.309 effort=1.4 velocity=12.5 -> lower=-1.309 upper=1.309 effort=112 velocity=12.5
- joint left_tarsus_joint: limit lower=-0.8779 upper=1.2497 effort=0 velocity=20 -> lower=-0.8779 upper=1.2497 effort=0.001 velocity=20
- joint left_toe_A_joint: limit lower=-0.912807183222 upper=1.2644910215 effort=0.9 velocity=11.5 -> lower=-0.912807183222 upper=1.2644910215 effort=45 velocity=11.5
- joint left_toe_B_joint: limit lower=-0.912807183222 upper=1.2644910215 effort=0.9 velocity=11.5 -> lower=-0.912807183222 upper=1.2644910215 effort=45 velocity=11.5
- joint left_toe_pitch_joint: limit lower=-0.785398163397 upper=0.785398163397 effort=0.9 velocity=11.5 -> lower=-0.785398163397 upper=0.785398163397 effort=0.001 velocity=11.5
- joint left_toe_roll_joint: limit lower=-0.6109 upper=0.6109 effort=0.9 velocity=11.5 -> lower=-0.6109 upper=0.6109 effort=0.001 velocity=11.5
- joint right_elbow_joint: limit lower=-1.3526 upper=1.3526 effort=1.4 velocity=12.5 -> lower=-1.3526 upper=1.3526 effort=112 velocity=12.5
- joint right_hip_pitch_joint: limit lower=-1.0472 upper=1.57079632679 effort=12.5 velocity=8.5 -> lower=-1.0472 upper=1.57079632679 effort=200 velocity=8.5
- joint right_hip_roll_joint: limit lower=-1.0472 upper=1.0472 effort=1.4 velocity=12.15 -> lower=-1.0472 upper=1.0472 effort=112 velocity=12.15
- joint right_hip_yaw_joint: limit lower=-0.698132 upper=0.698132 effort=1.4 velocity=12.15 -> lower=-0.698132 upper=0.698132 effort=70 velocity=12.15
- joint right_knee_joint: limit lower=-0.8727 upper=1.2392 effort=12.5 velocity=8.5085 -> lower=-0.8727 upper=1.2392 effort=200 velocity=8.5085
- joint right_shoulder_pitch_joint: limit lower=-2.5307 upper=2.5307 effort=1.4 velocity=12.5 -> lower=-2.5307 upper=2.5307 effort=112 velocity=12.5
- joint right_shoulder_roll_joint: limit lower=-1.309 upper=1.309 effort=1.4 velocity=12.5 -> lower=-1.309 upper=1.309 effort=112 velocity=12.5
- joint right_tarsus_joint: limit lower=-1.2497 upper=0.8779 effort=0 velocity=20 -> lower=-1.2497 upper=0.8779 effort=0.001 velocity=20
- joint right_toe_A_joint: limit lower=-1.2644910215 upper=0.912807183222 effort=0.9 velocity=11.5 -> lower=-1.2644910215 upper=0.912807183222 effort=45 velocity=11.5
- joint right_toe_B_joint: limit lower=-0.912807183222 upper=1.2644910215 effort=0.9 velocity=11.5 -> lower=-0.912807183222 upper=1.2644910215 effort=45 velocity=11.5
- joint right_toe_pitch_joint: limit lower=-0.785398163397 upper=0.785398163397 effort=0.9 velocity=11.5 -> lower=-0.785398163397 upper=0.785398163397 effort=0.001 velocity=11.5
- joint right_toe_roll_joint: limit lower=-0.6109 upper=0.6109 effort=0.9 velocity=11.5 -> lower=-0.6109 upper=0.6109 effort=0.0 velocity=11.5
- joint shoulder_yaw_joint_left: limit lower=-1.7453 upper=1.7453 effort=1.4 velocity=10 -> lower=-1.7453 upper=1.7453 effort=70 velocity=10
- joint shoulder_yaw_joint_right: limit lower=-1.7453 upper=1.7453 effort=1.4 velocity=10 -> lower=-1.7453 upper=1.7453 effort=70 velocity=10
