Commit message: add TSC_IMPL

File: Simulation/model/digit_model.urdf (robot description, URDF)
Before this commit: robot digit, 30 links, 29 joints
Links:
- removed link base
- added link contact1; visual box rgba=0 0 1 size=0.05 0.05 0.05
- added link contact2; visual box rgba=1 1 0 size=0.05 0.05 0.05
- added link contact3; visual box rgba=1 0 0 size=0.05 0.05 0.05
- added link contact4; visual box rgba=0 1 0 size=0.05 0.05 0.05
- added link contact5; visual box rgba=0 0 1 size=0.05 0.05 0.05
- added link contact6; visual box rgba=0 0 1 size=0.05 0.05 0.05
- added link contact7; visual box rgba=0 0 1 size=0.05 0.05 0.05
- added link contact8; visual box rgba=0 0 1 size=0.05 0.05 0.05
- link left_elbow: geometry collision mesh filename=package://digit_description//meshes/arm-L4.stl; visual mesh filename=package://digit_description//meshes/arm-L4.stl
- link left_hip_pitch: geometry collision mesh filename=package://digit_description//meshes/hip-pitch.stl; visual mesh filename=package://digit_description//meshes/hip-pitch.stl
- link left_hip_roll: geometry collision mesh filename=package://digit_description//meshes/hip-yaw-housing.stl; visual mesh filename=package://digit_description//meshes/hip-yaw-housing.stl
- link left_hip_yaw: geometry collision mesh filename=package://digit_description//meshes/hip-pitch-housing.stl; visual mesh filename=package://digit_description//meshes/hip-pitch-housing.stl
- link left_knee: geometry collision mesh filename=package://digit_description//meshes/knee.stl; visual mesh filename=package://digit_description//meshes/knee.stl
- link left_shin: geometry collision mesh filename=package://digit_description//meshes/shin.stl; visual mesh filename=package://digit_description//meshes/shin.stl
- link left_shoulder_cap: geometry collision mesh filename=package://digit_description//meshes/shoulder-roll-housing.s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; visual mesh filename=package://digit_description//meshes/shoulder-roll-housing.s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
- link left_shoulder_pitch: geometry collision mesh filename=package://digit_description//meshes/arm-L2.stl; visual mesh filename=package://digit_description//meshes/arm-L2.stl
- link left_shoulder_roll: geometry collision mesh filename=package://digit_description//meshes/arm-L1.stl; visual mesh filename=package://digit_description//meshes/arm-L1.stl
- link left_shoulder_yaw: geometry collision mesh filename=package://digit_description//meshes/arm-L3.stl; visual mesh filename=package://digit_description//meshes/arm-L3.stl
- link left_tarsus: geometry collision mesh filename=package://digit_description//meshes/tarsus.stl; visual mesh filename=package://digit_description//meshes/tarsus.stl
- link left_toe_pitch: geometry collision mesh filename=package://digit_description//meshes/toe-pitch.stl; visual mesh filename=package://digit_description//meshes/toe-pitch.stl
- link left_toe_roll: geometry collision mesh filename=package://digit_description//meshes/toe-roll.stl; visual mesh filename=package://digit_description//meshes/toe-roll.stl
- link right_elbow: geometry collision mesh filename=package://digit_description//meshes/arm-L4.stl scale=1 -1 1; visual mesh filename=package://digit_description//meshes/arm-L4.stl scale=1 -1 1
- link right_hip_pitch: geometry collision mesh filename=package://digit_description//meshes/hip-pitch.stl scale=1 -1 1; visual mesh filename=package://digit_description//meshes/hip-pitch.stl scale=1 -1 1
- link right_hip_roll: geometry collision mesh filename=package://digit_description//meshes/hip-yaw-housing.stl scale=1 -1 1; visual mesh filename=package://digit_description//meshes/hip-yaw-housing.stl scale=1 -1 1
- link right_hip_yaw: geometry collision mesh filename=package://digit_description//meshes/hip-pitch-housing.stl scale=1 -1 1; visual mesh filename=package://digit_description//meshes/hip-pitch-housing.stl scale=1 -1 1
- link right_knee: geometry collision mesh filename=package://digit_description//meshes/knee.stl scale=1 -1 1; visual mesh filename=package://digit_description//meshes/knee.stl scale=1 -1 1
- link right_shin: geometry collision mesh filename=package://digit_description//meshes/shin.stl scale=1 -1 1; visual mesh filename=package://digit_description//meshes/shin.stl scale=1 -1 1
- link right_shoulder_cap: geometry collision mesh filename=package://digit_description//meshes/shoulder-roll-housing.s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 scale=1 -1 1; visual mesh filename=package://digit_description//meshes/shoulder-roll-housing.s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 scale=1 -1 1
- link right_shoulder_pitch: geometry collision mesh filename=package://digit_description//meshes/arm-L2.stl scale=1 -1 1; visual mesh filename=package://digit_description//meshes/arm-L2.stl scale=1 -1 1
- link right_shoulder_roll: geometry collision mesh filename=package://digit_description//meshes/arm-L1.stl scale=1 -1 1; visual mesh filename=package://digit_description//meshes/arm-L1.stl scale=1 -1 1
- link right_shoulder_yaw: geometry collision mesh filename=package://digit_description//meshes/arm-L3.stl scale=1 -1 1; visual mesh filename=package://digit_description//meshes/arm-L3.stl scale=1 -1 1
- link right_tarsus: geometry collision mesh filename=package://digit_description//meshes/tarsus.stl scale=1 -1 1; visual mesh filename=package://digit_description//meshes/tarsus.stl scale=1 -1 1
- link right_toe_pitch: geometry collision mesh filename=package://digit_description//meshes/toe-pitch.stl scale=1 -1 1; visual mesh filename=package://digit_description//meshes/toe-pitch.stl scale=1 -1 1
- link right_toe_roll: geometry collision mesh filename=package://digit_description//meshes/toe-roll.stl scale=1 -1 1; visual mesh filename=package://digit_description//meshes/toe-roll.stl scale=1 -1 1
- link torso: geometry collision mesh filename=package://digit_description//meshes/torso.stl; visual mesh filename=package://digit_description//meshes/torso.stl
Joints:
- removed joint floating_base
- added joint contact1_joint: type fixed, parent left_toe_roll, child contact1, origin xyz=0 0 0 rpy=0 0 0
- added joint contact2_joint: type fixed, parent left_toe_roll, child contact2, origin xyz=0 0 0 rpy=0 0 0
- added joint contact3_joint: type fixed, parent left_toe_roll, child contact3, origin xyz=0 0 0 rpy=0 0 0
- added joint contact4_joint: type fixed, parent left_toe_roll, child contact4, origin xyz=0 0 0 rpy=0 0 0
- added joint contact5_joint: type fixed, parent right_toe_roll, child contact5, origin xyz=0 0 0 rpy=0 0 0
- added joint contact6_joint: type fixed, parent right_toe_roll, child contact6, origin xyz=0 0 0 rpy=0 0 0
- added joint contact7_joint: type fixed, parent right_toe_roll, child contact7, origin xyz=0 0 0 rpy=0 0 0
- added joint contact8_joint: type fixed, parent right_toe_roll, child contact8, origin xyz=0 0 0 rpy=0 0 0
- joint elbow_joint_left: type continuous -> revolute
- joint elbow_joint_right: type continuous -> revolute
- joint hip_abduction_left: type continuous -> revolute
- joint hip_abduction_right: type continuous -> revolute
- joint hip_flexion_left: type continuous -> revolute
- joint hip_flexion_right: type continuous -> revolute
- joint hip_rotation_left: type continuous -> revolute
- joint hip_rotation_right: type continuous -> revolute
- joint knee_joint_left: type continuous -> revolute
- joint knee_joint_right: type continuous -> revolute
- joint shin_to_tarsus_left: type continuous -> revolute
- joint shin_to_tarsus_right: type continuous -> revolute
- joint shoulder_pitch_joint_left: type continuous -> revolute
- joint shoulder_pitch_joint_right: type continuous -> revolute
- joint shoulder_roll_joint_left: type continuous -> revolute
- joint shoulder_roll_joint_right: type continuous -> revolute
- joint shoulder_yaw_joint_left: type continuous -> revolute
- joint shoulder_yaw_joint_right: type continuous -> revolute
- joint toe_pitch_joint_left: type continuous -> revolute
- joint toe_pitch_joint_right: type continuous -> revolute
- joint toe_roll_joint_left: type continuous -> revolute
- joint toe_roll_joint_right: type continuous -> revolute

Commit message: normal closed chain but with no passive joints

File: Simulation/model/digit_model.urdf (robot description, URDF)
Before this commit: robot digit, 38 links, 37 joints
Joints:
- joint elbow_joint_left: limit lower=-1.3526 upper=1.3526 effort=1.4 velocity=12.5 -> lower=-1.3526 upper=1.3526 effort=112 velocity=12.5
- joint elbow_joint_right: limit lower=-1.3526 upper=1.3526 effort=1.4 velocity=12.5 -> lower=-1.3526 upper=1.3526 effort=112 velocity=12.5
- joint hip_abduction_left: limit lower=-1.0472 upper=1.0472 effort=1.4 velocity=12.15 -> lower=-1.0472 upper=1.0472 effort=112 velocity=12.15
- joint hip_abduction_right: limit lower=-1.0472 upper=1.0472 effort=1.4 velocity=12.15 -> lower=-1.0472 upper=1.0472 effort=112 velocity=12.15
- joint hip_flexion_left: limit lower=-1.0472 upper=1.57079632679 effort=12.5 velocity=8.5 -> lower=-1.0472 upper=1.57079632679 effort=200 velocity=8.5
- joint hip_flexion_right: limit lower=-1.57079632679 upper=1.0472 effort=12.5 velocity=8.5 -> lower=-1.57079632679 upper=1.0472 effort=200 velocity=8.5
- joint hip_rotation_left: limit lower=-0.698132 upper=0.698132 effort=1.4 velocity=12.15 -> lower=-0.698132 upper=0.698132 effort=70 velocity=12.15
- joint hip_rotation_right: limit lower=-0.698132 upper=0.698132 effort=1.4 velocity=12.15 -> lower=-0.698132 upper=0.698132 effort=70 velocity=12.15
- joint knee_joint_left: limit lower=-1.2392 upper=0.8727 effort=12.5 velocity=8.5085 -> lower=-1.2392 upper=0.8727 effort=200 velocity=8.5085
- joint knee_joint_right: limit lower=-0.8727 upper=1.2392 effort=12.5 velocity=8.5085 -> lower=-0.8727 upper=1.2392 effort=200 velocity=8.5085
- joint shin_to_tarsus_left: limit lower=-0.8779 upper=1.2497 effort=0 velocity=20 -> lower=-0.8779 upper=1.2497 effort=200 velocity=20
- joint shin_to_tarsus_right: limit lower=-1.2497 upper=0.8779 effort=0 velocity=20 -> lower=-1.2497 upper=0.8779 effort=200 velocity=20
- joint shoulder_pitch_joint_left: limit lower=-2.5307 upper=2.5307 effort=1.4 velocity=12.5 -> lower=-2.5307 upper=2.5307 effort=112 velocity=12.5
- joint shoulder_pitch_joint_right: limit lower=-2.5307 upper=2.5307 effort=1.4 velocity=12.5 -> lower=-2.5307 upper=2.5307 effort=112 velocity=12.5
- joint shoulder_roll_joint_left: limit lower=-1.309 upper=1.309 effort=1.4 velocity=12.5 -> lower=-1.309 upper=1.309 effort=112 velocity=12.5
- joint shoulder_roll_joint_right: limit lower=-1.309 upper=1.309 effort=1.4 velocity=12.5 -> lower=-1.309 upper=1.309 effort=112 velocity=12.5
- joint shoulder_yaw_joint_left: limit lower=-1.7453 upper=1.7453 effort=1.4 velocity=10 -> lower=-1.7453 upper=1.7453 effort=70 velocity=10
- joint shoulder_yaw_joint_right: limit lower=-1.7453 upper=1.7453 effort=1.4 velocity=10 -> lower=-1.7453 upper=1.7453 effort=70 velocity=10
- joint toe_pitch_joint_left: limit lower=-0.785398163397 upper=0.785398163397 effort=0.9 velocity=11.5 -> lower=-0.785398163397 upper=0.785398163397 effort=45 velocity=11.5
- joint toe_pitch_joint_right: limit lower=-0.785398163397 upper=0.785398163397 effort=0.9 velocity=11.5 -> lower=-0.785398163397 upper=0.785398163397 effort=45 velocity=11.5
- joint toe_roll_joint_left: limit lower=-0.6109 upper=0.6109 effort=0.9 velocity=11.5 -> lower=-0.6109 upper=0.6109 effort=45 velocity=11.5
- joint toe_roll_joint_right: limit lower=-0.6109 upper=0.6109 effort=0.9 velocity=11.5 -> lower=-0.6109 upper=0.6109 effort=45 velocity=11.5
