Commit message: add spring joints but has some problems

File: Simulation/model/digit_ysp_o.urdf (robot description, URDF)
Before this commit: robot digit, 61 links, 60 joints
Joints:
- joint left_heel_spring_joint: limit lower=-0.104719753333 upper=0.104719753333 effort=0.9 velocity=11.5 -> lower=-0.104719753333 upper=0.104719753333 effort=0.001 velocity=11.5; type fixed -> revolute
- joint left_shin_joint: limit lower=-0.35 upper=0.35 effort=0 velocity=10 -> lower=-0.35 upper=0.35 effort=0.001 velocity=10; type fixed -> revolute
- joint right_heel_spring_joint: limit lower=-0.104719753333 upper=0.104719753333 effort=0.9 velocity=11.5 -> lower=-0.104719753333 upper=0.104719753333 effort=0.001 velocity=11.5; type fixed -> revolute
- joint right_shin_joint: limit lower=-0.35 upper=0.35 effort=0 velocity=10 -> lower=-0.35 upper=0.35 effort=0.001 velocity=10; type fixed -> revolute

Commit message: with spring joints in simulation but not in controller model (not work)

File: Simulation/model/digit_ysp_o.urdf (robot description, URDF)
Before this commit: robot digit, 61 links, 60 joints
Joints:
- joint left_heel_spring_joint: type revolute -> fixed
- joint left_shin_joint: type revolute -> fixed
- joint right_heel_spring_joint: type revolute -> fixed
- joint right_shin_joint: type revolute -> fixed

Commit message: not work with spring joints

File: Simulation/model/digit_ysp_o.urdf (robot description, URDF)
Before this commit: robot digit, 61 links, 60 joints
Joints:
- joint left_heel_spring_joint: type fixed -> revolute
- joint left_shin_joint: type fixed -> revolute
- joint right_heel_spring_joint: type fixed -> revolute
- joint right_shin_joint: type fixed -> revolute
