Commit message: final version for control not include planning

File: digit_description/urdf/digit.urdf (robot description, URDF)
Before this commit: robot digit, 38 links, 37 joints
Links:
- removed link vectorNav
- added link cp_left_achillies_rod; visual sphere radius=0.010
- added link cp_left_heel_spring; visual sphere radius=0.015
- added link cp_left_toe_A_rod; visual sphere radius=0.010
- added link cp_left_toe_B_rod; visual sphere radius=0.010
- added link cp_left_toe_roll_A; visual sphere radius=0.015
- added link cp_left_toe_roll_B; visual sphere radius=0.015
- added link cp_right_achillies_rod; visual sphere radius=0.010
- added link cp_right_heel_spring; visual sphere radius=0.015
- added link cp_right_toe_A_rod; visual sphere radius=0.010
- added link cp_right_toe_B_rod; visual sphere radius=0.010
- added link cp_right_toe_roll_A; visual sphere radius=0.015
- added link cp_right_toe_roll_B; visual sphere radius=0.015
- added link left_achillies_rod, mass 0.178148; collision mesh filename=package://digit_description//meshes_new/achilles-rod.stl; visual mesh filename=package://digit_description//meshes_new/achilles-rod.stl
- added link left_heel_spring, mass 0.230018; collision mesh filename=package://digit_description//meshes_new/heel-spring.stl; visual mesh filename=package://digit_description//meshes_new/heel-spring.stl
- added link left_toe_A, mass 0.139557; collision mesh filename=package://digit_description//meshes_new/toe-output.stl; visual mesh filename=package://digit_description//meshes_new/toe-output.stl
- added link left_toe_A_rod, mass 0.090983; collision mesh filename=package://digit_description//meshes_new/toe-A-rod.stl; visual mesh filename=package://digit_description//meshes_new/toe-A-rod.stl
- added link left_toe_B, mass 0.139557; collision mesh filename=package://digit_description//meshes_new/toe-output.stl; visual mesh filename=package://digit_description//meshes_new/toe-output.stl
- added link left_toe_B_rod, mass 0.079507; collision mesh filename=package://digit_description//meshes_new/toe-B-rod.stl; visual mesh filename=package://digit_description//meshes_new/toe-B-rod.stl
- added link right_achillies_rod, mass 0.178148; collision mesh filename=package://digit_description//meshes_new/achilles-rod.stl scale=1 -1 1; visual mesh filename=package://digit_description//meshes_new/achilles-rod.stl scale=1 -1 1
- added link right_heel_spring, mass 0.230018; collision mesh filename=package://digit_description//meshes_new/heel-spring.stl scale=1 -1 1; visual mesh filename=package://digit_description//meshes_new/heel-spring.stl scale=1 -1 1
- added link right_toe_A, mass 0.139557; collision mesh filename=package://digit_description//meshes_new/toe-output.stl scale=1 -1 1; visual mesh filename=package://digit_description//meshes_new/toe-output.stl scale=1 -1 1
- added link right_toe_A_rod, mass 0.090983; collision mesh filename=package://digit_description//meshes_new/toe-A-rod.stl scale=1 -1 1; visual mesh filename=package://digit_description//meshes_new/toe-A-rod.stl scale=1 -1 1
- added link right_toe_B, mass 0.139557; collision mesh filename=package://digit_description//meshes_new/toe-output.stl scale=1 -1 1; visual mesh filename=package://digit_description//meshes_new/toe-output.stl scale=1 -1 1
- added link right_toe_B_rod, mass 0.079507; collision mesh filename=package://digit_description//meshes_new/toe-B-rod.stl scale=1 -1 1; visual mesh filename=package://digit_description//meshes_new/toe-B-rod.stl scale=1 -1 1
- link contact1: geometry visual sphere radius=0.015
- link contact2: geometry visual sphere radius=0.015
- link contact3: geometry visual sphere radius=0.015
- link contact4: geometry visual sphere radius=0.015
- link contact5: geometry visual sphere radius=0.015
- link contact6: geometry visual sphere radius=0.015
- link contact7: geometry visual sphere radius=0.015
- link contact8: geometry visual sphere radius=0.015
- link left_elbow: geometry collision mesh filename=package://digit_description//meshes_new/arm-L4.stl; visual mesh filename=package://digit_description//meshes_new/arm-L4.stl
- link left_hip_pitch: geometry collision mesh filename=package://digit_description//meshes_new/hip-pitch.stl; visual mesh filename=package://digit_description//meshes_new/hip-pitch.stl
- link left_hip_roll: geometry collision mesh filename=package://digit_description//meshes_new/hip-yaw-housing.stl; visual mesh filename=package://digit_description//meshes_new/hip-yaw-housing.stl
- link left_hip_yaw: geometry collision mesh filename=package://digit_description//meshes_new/hip-pitch-housing.s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; visual mesh filename=package://digit_description//meshes_new/hip-pitch-housing.s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
- link left_knee: geometry collision mesh filename=package://digit_description//meshes_new/knee.stl; visual mesh filename=package://digit_description//meshes_new/knee.stl
- link left_shin: geometry collision mesh filename=package://digit_description//meshes_new/shin.stl; visual mesh filename=package://digit_description//meshes_new/shin.stl
- link left_shoulder_cap: geometry collision mesh filename=package://digit_description//meshes_new/shoulder-roll-housi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; visual mesh filename=package://digit_description//meshes_new/shoulder-roll-housi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
- link left_shoulder_pitch: geometry collision mesh filename=package://digit_description//meshes_new/arm-L2.stl; visual mesh filename=package://digit_description//meshes_new/arm-L2.stl
- link left_shoulder_roll: geometry collision mesh filename=package://digit_description//meshes_new/arm-L1.stl; visual mesh filename=package://digit_description//meshes_new/arm-L1.stl
- link left_shoulder_yaw: geometry collision mesh filename=package://digit_description//meshes_new/arm-L3.stl; visual mesh filename=package://digit_description//meshes_new/arm-L3.stl
- link left_tarsus: geometry collision mesh filename=package://digit_description//meshes_new/tarsus.stl; visual mesh filename=package://digit_description//meshes_new/tarsus.stl
- link left_toe_pitch: geometry collision mesh filename=package://digit_description//meshes_new/toe-pitch.stl; visual mesh filename=package://digit_description//meshes_new/toe-pitch.stl
- link left_toe_roll: geometry collision mesh filename=package://digit_description//meshes_new/toe-roll.stl; visual mesh filename=package://digit_description//meshes_new/toe-roll.stl
- link left_waist_cap: geometry collision mesh filename=package://digit_description//meshes_new/shoulder-roll-housi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 scale=1 -1 1; visual mesh filename=package://digit_description//meshes_new/shoulder-roll-housi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 scale=1 -1 1
- link right_elbow: geometry collision mesh filename=package://digit_description//meshes_new/arm-L4.stl scale=1 -1 1; visual mesh filename=package://digit_description//meshes_new/arm-L4.stl scale=1 -1 1
- link right_hip_pitch: geometry collision mesh filename=package://digit_description//meshes_new/hip-pitch.stl scale=1 -1 1; visual mesh filename=package://digit_description//meshes_new/hip-pitch.stl scale=1 -1 1
- link right_hip_roll: geometry collision mesh filename=package://digit_description//meshes_new/hip-yaw-housing.stl scale=1 -1 1; visual mesh filename=package://digit_description//meshes_new/hip-yaw-housing.stl scale=1 -1 1
- link right_hip_yaw: geometry collision mesh filename=package://digit_description//meshes_new/hip-pitch-housing.s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 scale=1 -1 1; visual mesh filename=package://digit_description//meshes_new/hip-pitch-housing.s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 scale=1 -1 1
- link right_knee: geometry collision mesh filename=package://digit_description//meshes_new/knee.stl scale=1 -1 1; visual mesh filename=package://digit_description//meshes_new/knee.stl scale=1 -1 1
- link right_shin: geometry collision mesh filename=package://digit_description//meshes_new/shin.stl scale=1 -1 1; visual mesh filename=package://digit_description//meshes_new/shin.stl scale=1 -1 1
- link right_shoulder_cap: geometry collision mesh filename=package://digit_description//meshes_new/shoulder-roll-housi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 scale=1 -1 1; visual mesh filename=package://digit_description//meshes_new/shoulder-roll-housi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 scale=1 -1 1
- link right_shoulder_pitch: geometry collision mesh filename=package://digit_description//meshes_new/arm-L2.stl scale=1 -1 1; visual mesh filename=package://digit_description//meshes_new/arm-L2.stl scale=1 -1 1
- link right_shoulder_roll: geometry collision mesh filename=package://digit_description//meshes_new/arm-L1.stl scale=1 -1 1; visual mesh filename=package://digit_description//meshes_new/arm-L1.stl scale=1 -1 1
- link right_shoulder_yaw: geometry collision mesh filename=package://digit_description//meshes_new/arm-L3.stl scale=1 -1 1; visual mesh filename=package://digit_description//meshes_new/arm-L3.stl scale=1 -1 1
- link right_tarsus: geometry collision mesh filename=package://digit_description//meshes_new/tarsus.stl scale=1 -1 1; visual mesh filename=package://digit_description//meshes_new/tarsus.stl scale=1 -1 1
- link right_toe_pitch: geometry collision mesh filename=package://digit_description//meshes_new/toe-pitch.stl scale=1 -1 1; visual mesh filename=package://digit_description//meshes_new/toe-pitch.stl scale=1 -1 1
- link right_toe_roll: geometry collision mesh filename=package://digit_description//meshes_new/toe-roll.stl scale=1 -1 1; visual mesh filename=package://digit_description//meshes_new/toe-roll.stl scale=1 -1 1
- link right_waist_cap: geometry collision mesh filename=package://digit_description//meshes_new/shoulder-roll-housi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; visual mesh filename=package://digit_description//meshes_new/shoulder-roll-housi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
- link torso: geometry collision mesh filename=package://digit_description//meshes_new/torso.stl; visual mesh filename=package://digit_description//meshes_new/torso.stl
Joints:
- removed joint elbow_joint_left
- removed joint elbow_joint_right
- removed joint fixed_pelvis_to_vectorNav
- removed joint hip_abduction_left
- removed joint hip_abduction_right
- removed joint hip_flexion_left
- removed joint hip_flexion_right
- removed joint hip_rotation_left
- removed joint hip_rotation_right
- removed joint knee_joint_left
- removed joint knee_joint_right
- removed joint knee_to_shin_left
- removed joint knee_to_shin_right
- removed joint shin_to_tarsus_left
- removed joint shin_to_tarsus_right
- removed joint shoulder_cap_joint_right
- removed joint shoulder_pitch_joint_left
- removed joint shoulder_pitch_joint_right
- removed joint shoulder_roll_cap_left
- removed joint shoulder_roll_joint_left
- removed joint shoulder_roll_joint_right
- removed joint toe_pitch_joint_left
- removed joint toe_pitch_joint_right
- removed joint toe_roll_joint_left
- removed joint toe_roll_joint_right
- removed joint waist_cap_joint_left
- removed joint waist_cap_joint_right
- added joint cp_left_achillies_rod_joint: type fixed, parent left_achillies_rod, child cp_left_achillies_rod, origin xyz=0 0 0 rpy=0 0 0, axis 0 0 1
- added joint cp_left_heel_spring_joint: type fixed, parent left_heel_spring, child cp_left_heel_spring, origin xyz=0.113789 -0.011056 0 rpy=0 0 0, axis 0 0 1
- added joint cp_left_toe_A_rod_joint: type fixed, parent left_toe_A_rod, child cp_left_toe_A_rod, origin xyz=0 0 0 rpy=0 0 0, axis 0 0 1
- added joint cp_left_toe_B_rod_joint: type fixed, parent left_toe_B_rod, child cp_left_toe_B_rod, origin xyz=0 0 0 rpy=0 0 0, axis 0 0 1
- added joint cp_left_toe_roll_A_joint: type fixed, parent left_toe_roll, child cp_left_toe_roll_A, origin xyz=0.0179 -0.009551 -0.054164 rpy=0 0 0, axis 0 0 1
- added joint cp_left_toe_roll_B_joint: type fixed, parent left_toe_roll, child cp_left_toe_roll_B, origin xyz=-0.0181 -0.009551 -0.054164 rpy=0 0 0, axis 0 0 1
- added joint cp_right_achillies_rod_joint: type fixed, parent right_achillies_rod, child cp_right_achillies_rod, origin xyz=0 0 0 rpy=0 0 0, axis 0 0 1
- added joint cp_right_heel_spring_joint: type fixed, parent right_heel_spring, child cp_right_heel_spring, origin xyz=0.113789 0.011056 0 rpy=0 0 0, axis 0 0 1
- added joint cp_right_toe_A_rod_joint: type fixed, parent right_toe_A_rod, child cp_right_toe_A_rod, origin xyz=0 0 0 rpy=0 0 0, axis 0 0 1
- added joint cp_right_toe_B_rod_joint: type fixed, parent right_toe_B_rod, child cp_right_toe_B_rod, origin xyz=0 0 0 rpy=0 0 0, axis 0 0 1
- added joint cp_right_toe_roll_A_joint: type fixed, parent right_toe_roll, child cp_right_toe_roll_A, origin xyz=0.0179 0.009551 -0.054164 rpy=0 0 0, axis 0 0 1
- added joint cp_right_toe_roll_B_joint: type fixed, parent right_toe_roll, child cp_right_toe_roll_B, origin xyz=-0.0181 0.009551 -0.054164 rpy=0 0 0, axis 0 0 1
- added joint left_achillies_rod_joint: type fixed, parent left_hip_pitch, child left_achillies_rod, origin xyz=0 0 0.046 rpy=0.0087529 0.0708516 -1.435541, axis 0 1 0, limit lower=-1.5 upper=1.5 effort=12.5 velocity=8.5085
- added joint left_elbow_joint: type revolute, parent left_shoulder_yaw, child left_elbow, origin xyz=0 -0.0385 0.185 rpy=1.57079632679 -0.3926991 0, axis 0 0 1, limit lower=-1.3526 upper=1.3526 effort=1.4 velocity=12.5
- added joint left_heel_spring_joint: type fixed, parent left_tarsus, child left_heel_spring, origin xyz=-0.01766 -0.029456 0.00104 rpy=-0.0689073 -0.0370354 2.7207176, axis 0 0 1, limit lower=-0.104719753333 upper=0.104719753333 effort=0.9 velocity=11.5
- added joint left_hip_pitch_joint: type revolute, parent left_hip_yaw, child left_hip_pitch, origin xyz=0 0.004 0.068 rpy=-1.57079632679 -0.7853981 3.1415927, axis 0 0 -1, limit lower=-1.0472 upper=1.57079632679 effort=12.5 velocity=8.5
- added joint left_hip_roll_joint: type revolute, parent torso, child left_hip_roll, origin xyz=-0.001 0.091 0 rpy=1.57079632679 -1.1955506 -1.57079632679, axis 0 0 1, limit lower=-1.0472 upper=1.0472 effort=1.4 velocity=12.15
- added joint left_hip_yaw_joint: type revolute, parent left_hip_roll, child left_hip_yaw, origin xyz=-0.0505 0 0.044 rpy=0 -1.57079632679 0, axis 0 0 1, limit lower=-0.698132 upper=0.698132 effort=1.4 velocity=12.15
- added joint left_knee_joint: type revolute, parent left_hip_pitch, child left_knee, origin xyz=0.12 0 0.0045 rpy=0 0 -1.57079632679, axis 0 0 1, limit lower=-1.2392 upper=0.8727 effort=12.5 velocity=8.5085
- added joint left_shin_joint: type fixed, parent left_knee, child left_shin, origin xyz=0.060677 0.047406 0 rpy=0 0 0, axis 0 0 1, limit lower=-0.35 upper=0.35 effort=0 velocity=10
- added joint left_shoulder_cap_joint: type fixed, parent torso, child left_shoulder_cap, origin xyz=0.001 0.12 0.4 rpy=-1.57079632679 -1.3962633 1.57079632679, axis 0 0 1, limit lower=-1.309 upper=1.309 effort=1.4 velocity=12.5
- added joint left_shoulder_pitch_joint: type revolute, parent left_shoulder_roll, child left_shoulder_pitch, origin xyz=-0.00017 -0.011055 0.0555 rpy=1.57079632679 0.785398163397 0.0, axis 0 0 -1, limit lower=-2.5307 upper=2.5307 effort=1.4 velocity=12.5
- added joint left_shoulder_roll_joint: type revolute, parent torso, child left_shoulder_roll, origin xyz=-0.001 0.12 0.4 rpy=-1.57079632679 -1.3962633 1.57079632679, axis 0 0 1, limit lower=-1.309 upper=1.309 effort=1.4 velocity=12.5
- added joint left_tarsus_joint: type revolute, parent left_shin, child left_tarsus, origin xyz=0.434759 0.02 0 rpy=0 0 1.7976891, axis 0 0 1, limit lower=-0.8779 upper=1.2497 effort=0 velocity=20
- added joint left_toe_A_joint: type revolute, parent left_tarsus, child left_toe_A, origin xyz=0.059 -0.034 -0.0276 rpy=3.1415927 0 -1.6050048, axis 0 0 1, limit lower=-0.912807183222 upper=1.2644910215 effort=0.9 velocity=11.5
- added joint left_toe_A_rod_parent_joint: type fixed, parent left_toe_A, child left_toe_A_rod, origin xyz=0.057 0 -0.008 rpy=-0.0374899 0.0049742 -1.5964351, axis 0 1 0, limit lower=-3.785398163397 upper=3.785398163397 effort=0.9 velocity=11.5
- added joint left_toe_B_joint: type revolute, parent left_tarsus, child left_toe_B, origin xyz=0.111 -0.034 0.0276 rpy=0 0 -1.6049813, axis 0 0 1, limit lower=-0.912807183222 upper=1.2644910215 effort=0.9 velocity=11.5
- added joint left_toe_B_rod_parent_joint: type fixed, parent left_toe_B, child left_toe_B_rod, origin xyz=0.057 0 -0.008 rpy=-0.0536482 0.0051326 1.5948474, axis 0 1 0, limit lower=-3.785398163397 upper=3.785398163397 effort=0.9 velocity=11.5
- added joint left_toe_pitch_joint: type revolute, parent left_tarsus, child left_toe_pitch, origin xyz=0.408 -0.04 0 rpy=0 0 1.1956, axis 0 0 1, limit lower=-0.785398163397 upper=0.785398163397 effort=0.9 velocity=11.5
- added joint left_toe_roll_joint: type revolute, parent left_toe_pitch, child left_toe_roll, origin xyz=0 0 0 rpy=0 1.57079632679 0, axis 0 0 1, limit lower=-0.6109 upper=0.6109 effort=0.9 velocity=11.5
- added joint left_waist_cap_joint: type fixed, parent torso, child left_waist_cap, origin xyz=-0.001 0.09 0.0 rpy=-1.57079632679 1.57 1.57079632679, axis 0 0 1, limit lower=-1.309 upper=1.309 effort=1.4 velocity=12.5
- added joint right_achillies_rod_joint: type fixed, parent right_hip_pitch, child right_achillies_rod, origin xyz=0 0 0.046 rpy=-0.0087529 0.0708516 1.435541, axis 0 1 0, limit lower=-1.5 upper=1.5 effort=12.5 velocity=8.5085
- added joint right_elbow_joint: type revolute, parent right_shoulder_yaw, child right_elbow, origin xyz=0 0.0385 0.185 rpy=-1.57079632679 -0.3926991 0, axis 0 0 1, limit lower=-1.3526 upper=1.3526 effort=1.4 velocity=12.5
- added joint right_heel_spring_joint: type fixed, parent right_tarsus, child right_heel_spring, origin xyz=-0.01766 0.029456 0.00104 rpy=0.0689073 -0.0370354 -2.7207176, axis 0 0 1, limit lower=-0.104719753333 upper=0.104719753333 effort=0.9 velocity=11.5
- added joint right_hip_pitch_joint: type revolute, parent right_hip_yaw, child right_hip_pitch, origin xyz=0 -0.004 0.068 rpy=1.57079632679 -0.7853981 -3.1415927, axis 0 0 -1, limit lower=-1.0472 upper=1.57079632679 effort=12.5 velocity=8.5
- added joint right_hip_roll_joint: type revolute, parent torso, child right_hip_roll, origin xyz=-0.001 -0.091 0 rpy=-1.57079632679 -1.1955506 1.57079632679, axis 0 0 1, limit lower=-1.0472 upper=1.0472 effort=1.4 velocity=12.15
- added joint right_hip_yaw_joint: type revolute, parent right_hip_roll, child right_hip_yaw, origin xyz=-0.0505 0 0.044 rpy=0 -1.57079632679 0, axis 0 0 1, limit lower=-0.698132 upper=0.698132 effort=1.4 velocity=12.15
- added joint right_knee_joint: type revolute, parent right_hip_pitch, child right_knee, origin xyz=0.12 0 0.0045 rpy=0 0 1.57079632679, axis 0 0 1, limit lower=-0.8727 upper=1.2392 effort=12.5 velocity=8.5085
- added joint right_shin_joint: type fixed, parent right_knee, child right_shin, origin xyz=0.060677 -0.047406 0 rpy=0 0 0, axis 0 0 1, limit lower=-0.35 upper=0.35 effort=0 velocity=10
- added joint right_shoulder_cap_joint: type fixed, parent torso, child right_shoulder_cap, origin xyz=0.001 -0.12 0.4 rpy=1.57079632679 -1.3962633 -1.57079632679, axis 0 0 1, limit lower=-1.309 upper=1.309 effort=1.4 velocity=12.5
- added joint right_shoulder_pitch_joint: type revolute, parent right_shoulder_roll, child right_shoulder_pitch, origin xyz=-0.00017 0.011055 0.0555 rpy=-1.57079632679 0.785398163397 0.0, axis 0 0 -1, limit lower=-2.5307 upper=2.5307 effort=1.4 velocity=12.5
- added joint right_shoulder_roll_joint: type revolute, parent torso, child right_shoulder_roll, origin xyz=-0.001 -0.12 0.4 rpy=1.57079632679 -1.3962633 -1.57079632679, axis 0 0 1, limit lower=-1.309 upper=1.309 effort=1.4 velocity=12.5
- added joint right_tarsus_joint: type revolute, parent right_shin, child right_tarsus, origin xyz=0.434759 -0.02 0 rpy=0 0 -1.7976891, axis 0 0 1, limit lower=-1.2497 upper=0.8779 effort=0 velocity=20
- added joint right_toe_A_joint: type revolute, parent right_tarsus, child right_toe_A, origin xyz=0.059 0.034 -0.0276 rpy=-3.1415927 0 1.6050048, axis 0 0 1, limit lower=-1.2644910215 upper=0.912807183222 effort=0.9 velocity=11.5
- added joint right_toe_A_rod_parent_joint: type fixed, parent right_toe_A, child right_toe_A_rod, origin xyz=0.057 0 -0.008 rpy=0.0374899 0.0049742 1.5964351, axis 0 1 0, limit lower=-3.785398163397 upper=3.785398163397 effort=0.9 velocity=11.5
- added joint right_toe_B_joint: type revolute, parent right_tarsus, child right_toe_B, origin xyz=0.111 0.034 0.0276 rpy=0 0 1.6049813, axis 0 0 1, limit lower=-0.912807183222 upper=1.2644910215 effort=0.9 velocity=11.5
- added joint right_toe_B_rod_parent_joint: type fixed, parent right_toe_B, child right_toe_B_rod, origin xyz=0.057 0 -0.008 rpy=0.0536482 0.0051326 -1.5948474, axis 0 1 0, limit lower=-3.785398163397 upper=3.785398163397 effort=0.9 velocity=11.5
- added joint right_toe_pitch_joint: type revolute, parent right_tarsus, child right_toe_pitch, origin xyz=0.408 0.04 0 rpy=0 0 -1.1956, axis 0 0 1, limit lower=-0.785398163397 upper=0.785398163397 effort=0.9 velocity=11.5
- added joint right_toe_roll_joint: type revolute, parent right_toe_pitch, child right_toe_roll, origin xyz=0 0 0 rpy=0 1.57079632679 0, axis 0 0 1, limit lower=-0.6109 upper=0.6109 effort=0.9 velocity=11.5
- added joint right_waist_cap_joint: type fixed, parent torso, child right_waist_cap, origin xyz=-0.001 -0.09 0.0 rpy=1.57079632679 1.57 -1.57079632679, axis 0 0 1, limit lower=-1.309 upper=1.309 effort=1.4 velocity=12.5
- joint contact1_joint: origin xyz=-0.04000014 -0.11085709 0.07003817 rpy=0 0 0 -> xyz=0 0 0 rpy=0 0 0
- joint contact2_joint: origin xyz=0.03999983 -0.11082681 0.07005585 rpy=0 0 0 -> xyz=0 0 0 rpy=0 0 0
- joint contact3_joint: origin xyz=-0.04000029 0.00799069 -0.13385178 rpy=0 0 0 -> xyz=0 0 0 rpy=0 0 0
- joint contact4_joint: origin xyz=0.03999968 0.00802097 -0.13383410 rpy=0 0 0 -> xyz=0 0 0 rpy=0 0 0
- joint contact5_joint: origin xyz=0.03999945 0.11063009 0.07017034 rpy=0 0 0 -> xyz=0 0 0 rpy=0 0 0
- joint contact6_joint: origin xyz=-0.04000014 0.11085020 0.07004217 rpy=0 0 0 -> xyz=0 0 0 rpy=0 0 0
- joint contact7_joint: origin xyz=0.03999968 -0.00801787 -0.13383595 rpy=0 0 0 -> xyz=0 0 0 rpy=0 0 0
- joint contact8_joint: origin xyz=-0.04000029 -0.00798741 -0.13385373 rpy=0 0 0 -> xyz=0 0 0 rpy=0 0 0
